File: KICAD/CM400T_CDI_Revision_C/CM400T_CDI_Revision_C.kicad_pcb (KiCad board)
At the start: 2 copper layers, 70.4 x 40 mm, 41 parts

Commit message: Redraw schematic to match structure of diagram from manual. No electrical / functional changes
Parts:
- renumbered BR to P1, GC to P2, BW to P3, Y to P4, BL to P5, WH to P6, LB to P7, GH to P8, PI to P9
Connections:
- net Net-(C1-Pad1) renamed /Coil Output +
- net Net-(C1-Pad2) renamed /Main Cap +
- net Net-(C3-Pad1) renamed /Fixed Pulse
- net Net-(C3-Pad2) renamed GND
- net Net-(D1-Pad1) renamed /Ignition Winding -
- net Net-(D5-Pad1) renamed /SCR Gate
- net Net-(D6-Pad2) renamed /Spark Advance Pulse
- net Net-(D7-Pad1) renamed /Fixed Pulse Limiter
- net Net-(D8-Pad2) renamed /Ignition Winding +
- net Net-(D9-Pad1) renamed /Kill Switch

Commit message: Add footprint file for 35mm capacitor to fix DRC violation
Parts:
- C1: footprint Capacitor_THT:C_Axial_L3.8mm_D2.6mm_P12.50mm_Horizontal -> footprints:C_Axial_L3.8mm_D2.6mm_P35.00mm_Horizontal
Changed lines of the file:
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@@
 		)
 	)
-	(footprint "Capacitor_THT:C_Axial_L3.8mm_D2.6mm_P12.50mm_Horizontal"
+	(footprint "footprints:C_Axial_L3.8mm_D2.6mm_P35.00mm_Horizontal"
 		(layer "F.Cu")
 		(at 116.1775 91.25)
-		(descr "C, Axial series, Axial, Horizontal, pin pitch=12.5mm, , length*diameter=3.8*2.6mm^2, http://www.vishay.com/docs/45231/arseries.pdf")
-		(tags "C Axial series Axial Horizontal pin pitch 12.5mm  length 3.8mm diameter 2.6mm")
+		(descr "C, Axial series, Axial, Horizontal, pin pitch=35mm, , length*diameter=3.8*2.6mm^2")
+		(tags "C Axial series Axial Horizontal pin pitch 35mm  length 3.8mm diameter 2.6mm")
 		(property "Reference" "C1"
 			(at 19.05 0 0)
@@
 		)
 		(embedded_fonts no)
-		(model "${KICAD6_3DMODEL_DIR}/Capacitor_THT.3dshapes/C_Axial_L3.8mm_D2.6mm_P12.50mm_Horizontal.wrl"
+		(model "${KICAD9_3DMODEL_DIR}/Capacitor_THT.3dshapes/CP_Axial_L29.0mm_D10.0mm_P35.00mm_Horizontal.wrl"
 			(offset
 				(xyz 0 0 0)

Commit message: Add ColorCode field to wire hole symbols so that code can be displayed on silkscreen instead of reference designator
Changed lines of the file:
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@@
 			(psa4output no)
 			(plot_black_and_white yes)
-			(plotinvisibletext no)
 			(sketchpadsonfab no)
 			(plotpadnumbers no)
@@
 			(at -2.752 0 90)
 			(layer "F.SilkS")
+			(hide yes)
 			(effects
 				(font
@@
 			)
 		)
+		(property "ColorCode" "BL"
+			(at -2.75 0 90)
+			(unlocked yes)
+			(layer "F.SilkS")
+			(effects
+				(font
+					(size 1 1)
+					(thickness 0.15)
+				)
+			)
+		)
 		(property ki_fp_filters "Pin* Test*")
 		(sheetname "/")
@@
 			(at -2.752 0 90)
 			(layer "F.SilkS")
+			(hide yes)
 			(effects
 				(font
@@
 			)
 		)
+		(property "ColorCode" "GH"
+			(at -2.752 0 90)
+			(unlocked yes)
+			(layer "F.SilkS")
+			(effects
+				(font
+					(size 1 1)
+					(thickness 0.15)
+				)
+			)
+		)
 		(property ki_fp_filters "Pin* Test*")
 		(sheetname "/")
@@
 			(at -2.752 0 90)
 			(layer "F.SilkS")
+			(hide yes)
 			(effects
 				(font
@@
 			)
 		)
+		(property "ColorCode" "WH"
+			(at -2.75 0 90)
+			(unlocked yes)
+			(layer "F.SilkS")
+			(effects
+				(font
+					(size 1 1)
+					(thickness 0.15)
+				)
+			)
+		)
 		(property ki_fp_filters "Pin* Test*")
 		(sheetname "/")
@@
 			(at -2.752 -0.5 90)
 			(layer "F.SilkS")
+			(hide yes)
 			(effects
 				(font
@@
 			)
 		)
+		(property "ColorCode" "LB"
+			(at -2.752 0 90)
+			(unlocked yes)
+			(layer "F.SilkS")
+			(effects
+				(font
+					(size 1 1)
+					(thickness 0.15)
+				)
+			)
+		)
 		(property ki_fp_filters "Pin* Test*")
 		(sheetname "/")
@@
 		(property "Reference" "P1"
 			(at -2.896 -0.248 90)
-			(layer "F.SilkS")
+			(layer "F.Fab")
 			(effects
 				(font
@@
 			)
 		)
+		(property "ColorCode" "BR"
+			(at -2.896 0 90)
+			(unlocked yes)
+			(layer "F.SilkS")
+			(effects
+				(font
+					(size 1 1)
+					(thickness 0.15)
+				)
+			)
+		)
 		(property ki_fp_filters "Pin* Test*")
 		(sheetname "/")
@@
 			(at -2.752 -0.5 90)
 			(layer "F.SilkS")
+			(hide yes)
 			(effects
 				(font
@@
 			)
 		)
+		(property "ColorCode" "Y"
+			(at -2.752 0 90)
+			(unlocked yes)
+			(layer "F.SilkS")
+			(effects
+				(font
+					(size 1 1)
+					(thickness 0.15)
+				)
+			)
+		)
 		(property ki_fp_filters "Pin* Test*")
 		(sheetname "/")
@@
 			(at -3 0 90)
 			(layer "F.SilkS")
+			(hide yes)
 			(effects
 				(font
@@
 			)
 		)
+		(property "ColorCode" "PI"
+			(at -3 0 90)
+			(unlocked yes)
+			(layer "F.SilkS")
+			(effects
+				(font
+					(size 1 1)
+					(thickness 0.15)
+				)
+			)
+		)
 		(property ki_fp_filters "Pin* Test*")
 		(sheetname "/")
@@
 			(at -2.752 0 90)
 			(layer "F.SilkS")
+			(hide yes)
 			(effects
 				(font
@@
 			)
 		)
+		(property "ColorCode" "BW"
+			(at -2.752 0 90)
+			(unlocked yes)
+			(layer "F.SilkS")
+			(effects
+				(font
+					(size 1 1)
+					(thickness 0.15)
+				)
+			)
+		)
 		(property ki_fp_filters "Pin* Test*")
 		(sheetname "/")
@@
 			(at -2.752 -0.248 90)
 			(layer "F.SilkS")
+			(hide yes)
 			(effects
 				(font
@@
 					(thickness 0.15)
 				)
+			)
+		)
+		(property "ColorCode" "GR"
+			(at -2.752 0 90)
+			(unlocked yes)
+			(layer "F.SilkS")
+			(effects
+				(font
+					(size 1 1)
+					(thickness 0.15)
+				)
